File: hardware/v2.0/flash.kicad_sch (KiCad schematic)
At the start: 10 parts, among them U1 ECP5-CABGA256, U12 W25Q128JVS

Commit message: Initial plan for adding an external ADC
Parts:
- U1: value ECP5-CABGA256 -> ECP5U-25F-CABGA256; LCSC Link https://lcsc.com/product-detail/Programmable-Logic-Device-C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 -> (none); LCSC Part # C1521614 -> (none); Manufactuer Part Number LFE5U-25F-6BG256C -> (none)
Changed lines of the file:
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@@
 			)
 		)
-		(property "Value" "ECP5-CABGA256"
+		(property "Value" "ECP5U-25F-CABGA256"
 			(at 117.602 121.412 0)
 			(effects
@@
 			(effects
 				(font
-					(size 1.27 1.27)
-				)
-				(hide yes)
-			)
-		)
-		(property "LCSC Link" "https://lcsc.com/product-detail/Programmable-Logic-Device-CPLDs-FPGAs_Lattice-LFE5U-25F-6BG256C_C1521614.html"
-			(at 111.76 110.49 0)
-			(effects
-				(font
-					(size 1.27 1.27)
-				)
-				(hide yes)
-			)
-		)
-		(property "Manufactuer Part Number" "LFE5U-25F-6BG256C"
-			(at 111.76 110.49 0)
-			(effects
-				(font
-					(size 1.27 1.27)
-				)
-				(hide yes)
-			)
-		)
-		(property "LCSC Part #" "C1521614"
-			(at 111.76 110.49 0)
-			(effects
-				(font
-					(size 1.27 1.27)
-				)
-				(hide yes)
-			)
-		)
-		(property "Note" ""
-			(at 111.76 110.49 0)
-			(effects
-				(font
-					(size 1.27 1.27)
-				)
-				(hide yes)
-			)
-		)
-		(property "Notes" ""
-			(at 111.76 110.49 0)
-			(effects
-				(font
