File: hardware/v2.0/flash.kicad_sch (KiCad schematic)
At the start: 10 parts, among them U1 ECP5U-25F-CABGA256, U12 W25Q128JVS

Commit message: Repo links update
Other:
- title: Icepi Zero -> GammaPi Zero
Changed lines of the file:
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@@
 	(paper "A4")
 	(title_block
-		(title "Icepi Zero")
-		(date "2026-01-17")
-		(rev "v2.1")
+		(title "GammaPi Zero")
+		(date "2026-01-25")
+		(rev "v2.3.2")
 		(company "Vadym Vikulin, Chengyin Yao (cheyao)")
-		(comment 1 "https://github.com/vikulin/icepi-zero")
+		(comment 1 "https://github.com/vikulin/gammapi-zero")
 		(comment 2 "License: Solderpad")
 		(comment 9 "OSHWA FR000026")
