File: hardware/v2.0/gpdi.kicad_sch (KiCad schematic)
At the start: 20 parts, among them J2 GPDI_C_1.3, U1 ECP5-CABGA256, U5 TPD2EUSB30A, U6 PCA9306DC1

Commit message: Initial plan for adding an external ADC
Parts:
- U1: value ECP5-CABGA256 -> ECP5U-25F-CABGA256; LCSC Link https://lcsc.com/product-detail/Programmable-Logic-Device-C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 -> (none); LCSC Part # C1521614 -> (none); Manufactuer Part Number LFE5U-25F-6BG256C -> (none)
Changed lines of the file:
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@@
 			)
 		)
-		(property "Value" "ECP5-CABGA256"
+		(property "Value" "ECP5U-25F-CABGA256"
 			(at 93.98 95.504 0)
 			(effects
@@
 			(effects
 				(font
-					(size 1.27 1.27)
-				)
-				(hide yes)
-			)
-		)
-		(property "LCSC Link" "https://lcsc.com/product-detail/Programmable-Logic-Device-CPLDs-FPGAs_Lattice-LFE5U-25F-6BG256C_C1521614.html"
-			(at 86.36 76.2 0)
-			(effects
-				(font
-					(size 1.27 1.27)
-				)
-				(hide yes)
-			)
-		)
-		(property "Manufactuer Part Number" "LFE5U-25F-6BG256C"
-			(at 86.36 76.2 0)
-			(effects
-				(font
-					(size 1.27 1.27)
-				)
-				(hide yes)
-			)
-		)
-		(property "LCSC Part #" "C1521614"
-			(at 86.36 76.2 0)
-			(effects
-				(font
-					(size 1.27 1.27)
-				)
-				(hide yes)
-			)
-		)
-		(property "Note" ""
-			(at 86.36 76.2 0)
-			(effects
-				(font
-					(size 1.27 1.27)
-				)
-				(hide yes)
-			)
-		)
-		(property "Notes" ""
-			(at 86.36 76.2 0)
-			(effects
-				(font
