File: hardware/v2.0/gpdi.kicad_sch (KiCad schematic)
At the start: 20 parts, among them J2 GPDI_C_1.3, U1 ECP5U-25F-CABGA256, U6 PCA9306DC1

Commit message: JLCPCB profile
Parts:
- U1: LCSC Part # (none) -> C1521614
Changed lines of the file:
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@@
 	(title_block
 		(title "GammaPi Zero")
-		(date "2026-02-08")
-		(rev "v2.7.0")
+		(date "2026-02-28")
+		(rev "v2.7.1")
 		(company "Vadym Vikulin, Chengyin Yao (cheyao)")
 		(comment 1 "https://github.com/vikulin/gammapi-zero")
@@
 			(at 86.36 76.2 0)
 			(effects
+				(font
+					(size 1.27 1.27)
+				)
+				(hide yes)
+			)
+		)
+		(property "LCSC Part #" "C1521614"
+			(at 86.36 76.2 0)
+			(effects
