File: hardware/v2.0/icepi-zero.kicad_sch (KiCad schematic)
At the start: 30 parts, among them J1 Conn_02x20_Counter_Clockwise, SW1 SW_Push, SW2 SW_Push, U1 ECP5U-25F-CABGA256, Y1 SG-8018CG 50.000000MHz

Commit message: LTC2630 DAC
Other:
- added sheet DAC (dac.kicad_sch)
Changed lines of the file:
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@@
 	)
 	(sheet
-		(at 200.152 54.61)
+		(at 206.502 54.61)
 		(size 17.78 10.16)
 		(exclude_from_sim no)
@@
 		)
 		(property "Sheetname" "Unused IO"
-			(at 200.152 53.8984 0)
+			(at 206.502 53.8984 0)
 			(effects
 				(font
@@
 		)
 		(property "Sheetfile" "io.kicad_sch"
-			(at 200.152 65.3546 0)
+			(at 206.502 65.3546 0)
 			(effects
 				(font
@@
 	)
 	(sheet
-		(at 130.81 54.61)
+		(at 137.16 54.61)
 		(size 17.78 10.16)
 		(exclude_from_sim no)
@@
 		)
 		(property "Sheetname" "SDRAM"
-			(at 130.81 53.8984 0)
+			(at 137.16 53.8984 0)
 			(effects
 				(font
@@
 		)
 		(property "Sheetfile" "sdram.kicad_sch"
-			(at 130.81 65.3546 0)
+			(at 137.16 65.3546 0)
 			(effects
 				(font
@@
 	)
 	(sheet
-		(at 60.96 54.61)
+		(at 20.32 54.61)
+		(size 17.78 10.16)
+		(exclude_from_sim no)
+		(in_bom yes)
+		(on_board yes)
+		(dnp no)
+		(fields_autoplaced yes)
+		(stroke
+			(width 0.1524)
+			(type solid)
+		)
+		(fill
+			(color 0 0 0 0.0000)
+		)
+		(property "Sheetname" "DAC"
+			(at 20.32 53.8984 0)
+			(effects
+				(font
+					(size 1.27 1.27)
+				)
+				(justify left bottom)
+			)
+		)
+		(property "Sheetfile" "dac.kicad_sch"
+			(at 20.32 65.3546 0)
+			(effects
+				(font
+					(size 1.27 1.27)
+				)
+				(justify left top)
+			)
+		)
+		(instances
+			(project "icepi-zero"
+				(path "/f88da08e-cf42-4d03-a08f-3f602fe6658d"
+					(page "10")
+				)
+			)
+		)
+	)
+	(sheet
+		(at 67.31 54.61)
 		(size 17.78 10.16)
 		(exclude_from_sim no)
@@
 		)
 		(property "Sheetname" "Power"
-			(at 60.96 53.8984 0)
+			(at 67.31 53.8984 0)
 			(effects
 				(font
@@
 		)
 		(property "Sheetfile" "power.kicad_sch"
-			(at 60.96 65.3546 0)
+			(at 67.31 65.3546 0)
 			(effects
 				(font
@@
 	)
 	(sheet
-		(at 38.1 54.61)
+		(at 44.45 54.61)
 		(size 16.51 10.16)
 		(exclude_from_sim no)
@@
 		)
 		(property "Sheetname" "ADC"
-			(at 38.1 53.8984 0)
+			(at 44.45 53.8984 0)
 			(effects
 				(font
@@
 		)
 		(property "Sheetfile" "adc.kicad_sch"
-			(at 38.1 65.3546 0)
+			(at 44.45 65.3546 0)
 			(effects
 				(font
@@
 	)
 	(sheet
-		(at 107.95 54.61)
+		(at 114.3 54.61)
 		(size 17.78 10.16)
 		(exclude_from_sim no)
@@
 		)
 		(property "Sheetname" "USB"
-			(at 107.95 53.8984 0)
+			(at 114.3 53.8984 0)
 			(effects
 				(font
@@
 		)
 		(property "Sheetfile" "usb.kicad_sch"
-			(at 107.95 65.3546 0)
+			(at 114.3 65.3546 0)
 			(effects
 				(font
@@
 	)
 	(sheet
-		(at 177.038 54.61)
+		(at 183.388 54.61)
 		(size 17.78 10.16)
 		(exclude_from_sim no)
@@
 		)
 		(property "Sheetname" "uSD"
-			(at 177.038 53.8984 0)
+			(at 183.388 53.8984 0)
 			(effects
 				(font
@@
 		)
 		(property "Sheetfile" "sd.kicad_sch"
-			(at 177.038 65.3546 0)
+			(at 183.388 65.3546 0)
 			(effects
 				(font
@@
 	)
 	(sheet
-		(at 153.67 54.61)
+		(at 160.02 54.61)
 		(size 17.78 10.16)
 		(exclude_from_sim no)
@@
 		)
 		(property "Sheetname" "Flash"
-			(at 153.67 53.8984 0)
+			(at 160.02 53.8984 0)
 			(effects
 				(font
@@
 		)
 		(property "Sheetfile" "flash.kicad_sch"
-			(at 153.67 65.3546 0)
+			(at 160.02 65.3546 0)
 			(effects
 				(font
@@
 	)
 	(sheet
-		(at 85.09 54.61)
+		(at 91.44 54.61)
 		(size 17.78 10.16)
 		(exclude_from_sim no)
@@
 		)
 		(property "Sheetname" "GPDI"
-			(at 85.09 53.8984 0)
+			(at 91.44 53.8984 0)
 			(effects
 				(font
@@
 		)
 		(property "Sheetfile" "gpdi.kicad_sch"
-			(at 85.09 65.3546 0)
-			(effects
-				(font
+			(at 91.44 65.3546 0)
+			(effects
+				(font

Commit message: DAC Vout
Connections:
- removed net ~{CS}(SPI): U1.C12 (PT56B/-)
Other:
- moved on the sheet: TP7, TP8

Commit message: Minor fixes
Other:
- note added: "Icepi Zero v2.5!"
- note removed: "Icepi Zero v2.0!"
Changed lines of the file:
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@@
 		(comment 9 "OSHWA FR000026")
 	)
-	(text "Icepi Zero v2.0!"
+	(text "Icepi Zero v2.5!"
 		(exclude_from_sim no)
 		(at 135.89 18.542 0)
