File: hardware/v2.0/sd.kicad_sch (KiCad schematic)
At the start: 3 parts, among them J6 Micro_SD_Card_Det2, U1 ECP5-CABGA256

Commit message: Initial plan for adding an external ADC
Parts:
- U1: value ECP5-CABGA256 -> ECP5U-25F-CABGA256; LCSC Link https://lcsc.com/product-detail/Programmable-Logic-Device-C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 -> (none); LCSC Part # C1521614 -> (none); Manufactuer Part Number LFE5U-25F-6BG256C -> (none)
Changed lines of the file:
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@@
 			)
 		)
-		(property "Value" "ECP5-CABGA256"
+		(property "Value" "ECP5U-25F-CABGA256"
 			(at 110.744 111.76 0)
 			(effects
@@
 			(effects
 				(font
-					(size 1.27 1.27)
-				)
-				(hide yes)
-			)
-		)
-		(property "LCSC Link" "https://lcsc.com/product-detail/Programmable-Logic-Device-CPLDs-FPGAs_Lattice-LFE5U-25F-6BG256C_C1521614.html"
-			(at 100.33 97.79 0)
-			(effects
-				(font
-					(size 1.27 1.27)
-				)
-				(hide yes)
-			)
-		)
-		(property "Manufactuer Part Number" "LFE5U-25F-6BG256C"
-			(at 100.33 97.79 0)
-			(effects
-				(font
-					(size 1.27 1.27)
-				)
-				(hide yes)
-			)
-		)
-		(property "LCSC Part #" "C1521614"
-			(at 100.33 97.79 0)
-			(effects
-				(font
-					(size 1.27 1.27)
-				)
-				(hide yes)
-			)
-		)
-		(property "Note" ""
-			(at 100.33 97.79 0)
-			(effects
-				(font
-					(size 1.27 1.27)
-				)
-				(hide yes)
-			)
-		)
-		(property "Notes" ""
-			(at 100.33 97.79 0)
-			(effects
-				(font
