File: hardware/v2.0/usb.kicad_sch (KiCad schematic)
At the start: 48 parts, among them J3 USB_C_Receptacle_USB2.0_14P, J4 USB_C_Receptacle_USB2.0_14P, J5 USB_C_Receptacle_USB2.0_14P, U1 ECP5-CABGA256, U10 TPD2EUSB30A, U7 TPD2EUSB30A, U8 TPD2EUSB30A, U9 FT231XQ

Commit message: Initial plan for adding an external ADC
Parts:
- U1: value ECP5-CABGA256 -> ECP5U-25F-CABGA256; LCSC Link https://lcsc.com/product-detail/Programmable-Logic-Device-C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 -> (none); LCSC Part # C1521614 -> (none); Manufactuer Part Number LFE5U-25F-6BG256C -> (none)
Changed lines of the file:
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@@
 			)
 		)
-		(property "Value" "ECP5-CABGA256"
+		(property "Value" "ECP5U-25F-CABGA256"
 			(at 189.992 141.478 0)
 			(effects
@@
 			)
 		)
-		(property "LCSC Link" "https://lcsc.com/product-detail/Programmable-Logic-Device-CPLDs-FPGAs_Lattice-LFE5U-25F-6BG256C_C1521614.html"
-			(at 198.12 132.08 0)
-			(effects
-				(font
-					(size 1.27 1.27)
-				)
-				(hide yes)
-			)
-		)
-		(property "Manufactuer Part Number" "LFE5U-25F-6BG256C"
-			(at 198.12 132.08 0)
-			(effects
-				(font
-					(size 1.27 1.27)
-				)
-				(hide yes)
-			)
-		)
-		(property "LCSC Part #" "C1521614"
-			(at 198.12 132.08 0)
-			(effects
-				(font
-					(size 1.27 1.27)
-				)
-				(hide yes)
-			)
-		)
-		(property "Note" ""
-			(at 198.12 132.08 0)
-			(effects
-				(font
-					(size 1.27 1.27)
-				)
-				(hide yes)
-			)
-		)
-		(property "Notes" ""
-			(at 198.12 132.08 0)
-			(effects
-				(font
-					(size 1.27 1.27)
-				)
-				(hide yes)
-			)
-		)
 		(pin "T2"
 		)
@@
 			)
 		)
-		(property "Value" "ECP5-CABGA256"
+		(property "Value" "ECP5U-25F-CABGA256"
 			(at 253.746 154.94 0)
 			(effects
@@
 			(effects
 				(font
-					(size 1.27 1.27)
-				)
-				(hide yes)
-			)
-		)
-		(property "LCSC Link" "https://lcsc.com/product-detail/Programmable-Logic-Device-CPLDs-FPGAs_Lattice-LFE5U-25F-6BG256C_C1521614.html"
-			(at 261.62 132.08 0)
-			(effects
-				(font
-					(size 1.27 1.27)
-				)
-				(hide yes)
-			)
-		)
-		(property "Manufactuer Part Number" "LFE5U-25F-6BG256C"
-			(at 261.62 132.08 0)
-			(effects
-				(font
-					(size 1.27 1.27)
-				)
-				(hide yes)
-			)
-		)
-		(property "LCSC Part #" "C1521614"
-			(at 261.62 132.08 0)
-			(effects
-				(font
-					(size 1.27 1.27)
-				)
-				(hide yes)
-			)
-		)
-		(property "Note" ""
-			(at 261.62 132.08 0)
-			(effects
-				(font
-					(size 1.27 1.27)
-				)
-				(hide yes)
-			)
-		)
-		(property "Notes" ""
-			(at 261.62 132.08 0)
-			(effects
-				(font
