File: hardware/v2.0/usb.kicad_sch (KiCad schematic)
At the start: 48 parts, among them J3 USB_C_Receptacle_USB2.0_14P, J4 USB_C_Receptacle_USB2.0_14P, J5 USB_C_Receptacle_USB2.0_14P, U1 ECP5U-25F-CABGA256, U10 TPD2EUSB30A, U7 TPD2EUSB30A, U8 TPD2EUSB30A, U9 FT231XQ

Commit message: Repo links update
Other:
- title: Icepi Zero -> GammaPi Zero
Changed lines of the file:
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@@
 	(paper "A4")
 	(title_block
-		(title "Icepi Zero")
-		(date "2026-01-17")
-		(rev "v2.1")
+		(title "GammaPi Zero")
+		(date "2026-01-25")
+		(rev "v2.3.2")
 		(company "Vadym Vikulin, Chengyin Yao (cheyao)")
-		(comment 1 "https://github.com/vikulin/icepi-zero")
+		(comment 1 "https://github.com/vikulin/gammapi-zero")
 		(comment 2 "License: Solderpad")
 		(comment 9 "OSHWA FR000026")
