File: hardware/v2.0/usb.kicad_sch (KiCad schematic)
At the start: 48 parts, among them J3 USB_C_Receptacle_USB2.0_14P, J4 USB_C_Receptacle_USB2.0_14P, J5 USB_C_Receptacle_USB2.0_14P, U1 ECP5U-25F-CABGA256, U10 TPD2EUSB30A, U7 TPD2EUSB30A, U8 TPD2EUSB30A, U9 FT231XQ

Commit message: JLCPCB profile
Parts:
- U1: LCSC Part # (none) -> C1521614
Changed lines of the file:
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@@
 	(title_block
 		(title "GammaPi Zero")
-		(date "2026-02-08")
-		(rev "v2.7.0")
+		(date "2026-02-28")
+		(rev "v2.7.1")
 		(company "Vadym Vikulin, Chengyin Yao (cheyao)")
 		(comment 1 "https://github.com/vikulin/gammapi-zero")
@@
 			)
 		)
+		(property "LCSC Part #" "C1521614"
+			(at 198.12 132.08 0)
+			(effects
+				(font
+					(size 1.27 1.27)
+				)
+				(hide yes)
+			)
+		)
 		(pin "T2"
 		)
@@
 			(at 261.62 132.08 0)
 			(effects
+				(font
+					(size 1.27 1.27)
+				)
+				(hide yes)
+			)
+		)
+		(property "LCSC Part #" "C1521614"
+			(at 261.62 132.08 0)
+			(effects
