File: hardware/v2.0/adc.kicad_sch (KiCad schematic)
At the start: 4 parts, among them IC2 LTC2256CUJ-12#PBF, U1 ECP5U-25F-CABGA256, Y2 SG-8018CG 50.000000MHz

Commit message: ADC CLKOUT±
Connections:
- net D6_7+: now also U1.M6 (PL47A/+/HS/LDQ44); no longer U1.N4 (PL38A/+/HS/LDQ44)
- net D6_7-: now also U1.N6 (PL47B/-/HS/LDQ44); no longer U1.P3 (PL38B/-/HS/LDQ44)
- net D8_9+: now also U1.N4 (PL38A/+/HS/LDQ44); no longer U1.L1 (PL26A/+/HS/LDQ32/PCLKT6_1)
- net D8_9-: now also U1.P3 (PL38B/-/HS/LDQ44); no longer U1.L2 (PL26B/-/HS/LDQ32/PCLKC6_1)
- net CLKOUT-: now reaches IC2.27 (CLKOUT-)
- net CLKOUT-: now also U1.L2 (PL26B/-/HS/LDQ32/PCLKC6_1)
- net CLKOUT+: now reaches IC2.28 (CLKOUT+)
- net CLKOUT+: now also U1.L1 (PL26A/+/HS/LDQ32/PCLKT6_1)
Other:
- company: Chengyin Yao (cheyao), Vadym Vikulin -> Vadym Vikulin, Chengyin Yao (cheyao)
- title: (none) -> Icepi Zero
Changed lines of the file:
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@@
 	(paper "A4")
 	(title_block
-		(date "2026-01-05")
-		(rev "v2.0")
-		(company "Chengyin Yao (cheyao), Vadym Vikulin")
+		(title "Icepi Zero")
+		(date "2026-01-17")
+		(rev "v2.1")
+		(company "Vadym Vikulin, Chengyin Yao (cheyao)")
+		(comment 1 "https://github.com/vikulin/icepi-zero")
+		(comment 2 "License: Solderpad")
+		(comment 9 "OSHWA FR000026")
 	)
 	(text "50MHz ADC Clock"
@@
 	(wire
 		(pts
+			(xy 220.472 57.15) (xy 239.522 57.15)
+		)
+		(stroke
+			(width 0)
+			(type default)
+		)
+	)
+	(wire
+		(pts
 			(xy 72.39 142.24) (xy 80.01 142.24)
 		)
@@
 	(wire
 		(pts
+			(xy 220.472 54.61) (xy 239.522 54.61)
+		)
+		(stroke
+			(width 0)
+			(type default)
+		)
+	)
+	(wire
+		(pts
 			(xy 138.43 92.71) (xy 157.48 92.71)
 		)
@@
 	(wire
 		(pts
+			(xy 78.74 91.44) (xy 97.79 91.44)
+		)
+		(stroke
+			(width 0)
+			(type default)
+		)
+	)
+	(wire
+		(pts
 			(xy 138.43 85.09) (xy 157.48 85.09)
+		)
+		(stroke
+			(width 0)
+			(type default)
+		)
+	)
+	(wire
+		(pts
+			(xy 78.74 93.98) (xy 97.79 93.98)
 		)
 		(stroke
@@
 		)
 	)
+	(label "CLKOUT+"
+		(at 231.14 54.61 180)
+		(effects
+			(font
+				(size 1.27 1.27)
+			)
+			(justify right bottom)
+		)
+	)
+	(label "CLKOUT-"
+		(at 97.79 91.44 180)
+		(effects
+			(font
+				(size 1.27 1.27)
+			)
+			(justify right bottom)
+		)
+	)
 	(label "D4_5-"
 		(at 138.43 69.85 0)
@@
 		)
 	)
+	(label "CLKOUT+"
+		(at 97.79 93.98 180)
+		(effects
+			(font
+				(size 1.27 1.27)
+			)
+			(justify right bottom)
+		)
+	)
 	(label "D4_5+"
 		(at 138.43 72.39 0)
@@
 	(label "D8_9-"
 		(at 157.48 85.09 180)
+		(effects
+			(font
+				(size 1.27 1.27)
+			)
+			(justify right bottom)
+		)
+	)
+	(label "CLKOUT-"
+		(at 231.14 57.15 180)
 		(effects
 			(font
@@
 		(pin "K5"
 		)
+		(pin "N6"
+		)
 		(instances

Commit message: ADC power
Parts:
- added C59: 2.2u, Capacitor_SMD:C_0603_1608Metric, symbol Device:C_Small
- added C60, C61, C66: 100n, Capacitor_SMD:C_0402_1005Metric, symbol Device:C
- added C64: 10uF, Capacitor_SMD:C_0603_1608Metric, symbol Device:C
- added C65: 1u, Capacitor_SMD:C_0402_1005Metric, symbol Device:C
- added FB2: 1k@100MHz, Inductor_SMD:L_0603_1608Metric, symbol Device:FerriteBead
- added R51: 100, Resistor_SMD:R_0402_1005Metric, symbol Device:R
Connections:
- net GND: now also IC2.25 (OGND), IC2.3 (GND_1), IC2.41 (GND_2), IC2.8 (PAR/~{SER}), C60.1, C61.1, C64.2, C65.2, C66.1
- net +1V8: now reaches IC2.10 (VDD_2)
- net +1V8: now also IC2.40 (VDD_3), IC2.9 (VDD_1), C64.1, FB2.1
- net FILTERED_1V8: now reaches IC2.26 (OVDD)
- net FILTERED_1V8: now also C65.1, C66.2, FB2.2
- net at IC2.35 (DNC_3): now also R51.1
- net at IC2.36 (OF): now also R51.2
- net at IC2.4 (REFH_1): now also IC2.5 (REFH_2), C59.1, C61.2
- net at IC2.6 (REFL_1): now also IC2.7 (REFL_2), C59.2, C60.2
- no-connect marks 0 -> 2

Commit message: ADC power
Parts:
- removed C64: 10uF, Capacitor_SMD:C_0603_1608Metric, symbol Device:C
- removed C65: 1u, Capacitor_SMD:C_0402_1005Metric, symbol Device:C
- removed C66: 100n, Capacitor_SMD:C_0402_1005Metric, symbol Device:C
- removed FB2: 1k@100MHz, Inductor_SMD:L_0603_1608Metric, symbol Device:FerriteBead
- added C67: 1u, Capacitor_SMD:C_0402_1005Metric, symbol Device:C
- added C68, C69: 100n, Capacitor_SMD:C_0402_1005Metric, symbol Device:C
- added R52: 100, Resistor_SMD:R_0402_1005Metric, symbol Device:R
Connections:
- net GND: now also C67.2, C68.1, C69.2
- net at IC2.37 (VCM): now also C68.2, R52.2
- net at IC2.38 (VREF): now also C67.1
- new net: C69.1, R52.1
Other:
- moved on the sheet: C55, Y2
