File: hardware/v2.0/sdram.kicad_sch (KiCad schematic)
At the start: 10 parts, among them IC1 IS42S16160J-6BLI, U1 ECP5U-25F-CABGA256

Commit message: BOM update
Parts:
- C46, C47, C48, C49, C50, C51, C52: footprint Capacitor_SMD:C_0603_1608Metric -> Capacitor_SMD:C_0402_1005Metric; MANUFACTURER_PART_NUMBER 0603B223K500NT -> 0402B223K500NT
Changed lines of the file:
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@@
 			)
 		)
-		(property "Footprint" "Capacitor_SMD:C_0603_1608Metric"
+		(property "Footprint" "Capacitor_SMD:C_0402_1005Metric"
 			(at 218.44 43.18 0)
 			(effects
@@
 			)
 		)
-		(property "Description" "Unpolarized capacitor, small symbol"
+		(property "Description" "22nF ±10% 50V Ceramic Capacitor X7R 0402"
 			(at 218.44 43.18 0)
 			(effects
@@
 			)
 		)
-		(property "MANUFACTURER_PART_NUMBER" "0603B223K500NT"
+		(property "MANUFACTURER_PART_NUMBER" "0402B223K500NT"
 			(at 218.44 43.18 0)
 			(effects
@@
 			)
 		)
-		(property "Footprint" "Capacitor_SMD:C_0603_1608Metric"
+		(property "Footprint" "Capacitor_SMD:C_0402_1005Metric"
 			(at 194.31 43.18 0)
 			(effects
@@
 			)
 		)
-		(property "Description" "Unpolarized capacitor, small symbol"
+		(property "Description" "22nF ±10% 50V Ceramic Capacitor X7R 0402"
 			(at 194.31 43.18 0)
 			(effects
@@
 			)
 		)
-		(property "MANUFACTURER_PART_NUMBER" "0603B223K500NT"
+		(property "MANUFACTURER_PART_NUMBER" "0402B223K500NT"
 			(at 194.31 43.18 0)
 			(effects
@@
 			)
 		)
-		(property "Footprint" "Capacitor_SMD:C_0603_1608Metric"
+		(property "Footprint" "Capacitor_SMD:C_0402_1005Metric"
 			(at 207.01 43.18 0)
 			(effects
@@
 			)
 		)
-		(property "Description" "Unpolarized capacitor, small symbol"
+		(property "Description" "22nF ±10% 50V Ceramic Capacitor X7R 0402"
 			(at 207.01 43.18 0)
 			(effects
@@
 			)
 		)
-		(property "MANUFACTURER_PART_NUMBER" "0603B223K500NT"
+		(property "MANUFACTURER_PART_NUMBER" "0402B223K500NT"
 			(at 207.01 43.18 0)
 			(effects
@@
 			)
 		)
-		(property "Footprint" "Capacitor_SMD:C_0603_1608Metric"
+		(property "Footprint" "Capacitor_SMD:C_0402_1005Metric"
 			(at 181.61 43.18 0)
 			(effects
@@
 			)
 		)
-		(property "Description" "Unpolarized capacitor, small symbol"
+		(property "Description" "22nF ±10% 50V Ceramic Capacitor X7R 0402"
 			(at 181.61 43.18 0)
 			(effects
@@
 			)
 		)
-		(property "MANUFACTURER_PART_NUMBER" "0603B223K500NT"
+		(property "MANUFACTURER_PART_NUMBER" "0402B223K500NT"
 			(at 181.61 43.18 0)
 			(effects
@@
 			)
 		)
-		(property "Footprint" "Capacitor_SMD:C_0603_1608Metric"
+		(property "Footprint" "Capacitor_SMD:C_0402_1005Metric"
 			(at 229.87 43.18 0)
 			(effects
@@
 			)
 		)
-		(property "Description" "Unpolarized capacitor, small symbol"
+		(property "Description" "22nF ±10% 50V Ceramic Capacitor X7R 0402"
 			(at 229.87 43.18 0)
 			(effects
@@
 			)
 		)
-		(property "MANUFACTURER_PART_NUMBER" "0603B223K500NT"
+		(property "MANUFACTURER_PART_NUMBER" "0402B223K500NT"
 			(at 229.87 43.18 0)
 			(effects
@@
 			)
 		)
-		(property "Footprint" "Capacitor_SMD:C_0603_1608Metric"
+		(property "Footprint" "Capacitor_SMD:C_0402_1005Metric"
 			(at 241.3 43.18 0)
 			(effects
@@
 			)
 		)
-		(property "Description" "Unpolarized capacitor, small symbol"
+		(property "Description" "22nF ±10% 50V Ceramic Capacitor X7R 0402"
 			(at 241.3 43.18 0)
 			(effects
@@
 			)
 		)
-		(property "MANUFACTURER_PART_NUMBER" "0603B223K500NT"
+		(property "MANUFACTURER_PART_NUMBER" "0402B223K500NT"
 			(at 241.3 43.18 0)
 			(effects
@@
 			)
 		)
-		(property "Footprint" "Capacitor_SMD:C_0603_1608Metric"
+		(property "Footprint" "Capacitor_SMD:C_0402_1005Metric"
 			(at 252.73 43.18 0)
 			(effects
@@
 			)
 		)
-		(property "Description" "Unpolarized capacitor, small symbol"
+		(property "Description" "22nF ±10% 50V Ceramic Capacitor X7R 0402"
 			(at 252.73 43.18 0)
 			(effects
@@
 			)
 		)
-		(property "MANUFACTURER_PART_NUMBER" "0603B223K500NT"
+		(property "MANUFACTURER_PART_NUMBER" "0402B223K500NT"
 			(at 252.73 43.18 0)
 			(effects
@@
 			)
 		)
-		(property "Description" "Unpolarized capacitor, small symbol"
+		(property "Description" "10uF ±10% 10V Ceramic Capacitor X5R 0603"
 			(at 264.16 43.18 0)
 			(effects
