File: hardware/v2.0/sdram.kicad_sch (KiCad schematic)
At the start: 10 parts, among them IC1 IS42S16160J-6BLI, U1 ECP5U-25F-CABGA256

Commit message: JLCPCB profile
Parts:
- C46, C47, C48, C49, C50, C51, C52: LCSC Part # C77571 -> C1532
- IC1: value IS42S16160J-6BLI -> IS42S16160J-6BLI-TR; LCSC Part # (none) -> C2063680
- U1: LCSC Part # (none) -> C1521614
Changed lines of the file:
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@@
 	(title_block
 		(title "GammaPi Zero")
-		(date "2026-02-08")
-		(rev "v2.7.0")
+		(date "2026-02-28")
+		(rev "v2.7.1")
 		(company "Vadym Vikulin, Chengyin Yao (cheyao)")
 		(comment 1 "https://github.com/vikulin/gammapi-zero")
@@
 			)
 		)
-		(property "LCSC Part #" "C77571"
+		(property "LCSC Part #" "C1532"
 			(at 218.44 43.18 0)
 			(effects
@@
 			)
 		)
-		(property "LCSC Part #" "C77571"
+		(property "LCSC Part #" "C1532"
 			(at 194.31 43.18 0)
 			(effects
@@
 			)
 		)
-		(property "LCSC Part #" "C77571"
+		(property "LCSC Part #" "C1532"
 			(at 207.01 43.18 0)
 			(effects
@@
 			)
 		)
-		(property "LCSC Part #" "C77571"
+		(property "LCSC Part #" "C1532"
 			(at 181.61 43.18 0)
 			(effects
@@
 			)
 		)
-		(property "LCSC Part #" "C77571"
+		(property "LCSC Part #" "C1532"
 			(at 229.87 43.18 0)
 			(effects
@@
 			)
 		)
-		(property "LCSC Part #" "C77571"
+		(property "LCSC Part #" "C1532"
 			(at 241.3 43.18 0)
 			(effects
@@
 			)
 		)
-		(property "LCSC Part #" "C77571"
+		(property "LCSC Part #" "C1532"
 			(at 252.73 43.18 0)
 			(effects
@@
 			)
 		)
+		(property "LCSC Part #" "C1521614"
+			(at 91.44 100.33 0)
+			(effects
+				(font
+					(size 1.27 1.27)
+				)
+				(hide yes)
+			)
+		)
 		(pin "T2"
 		)
@@
 			)
 		)
-		(property "Value" "IS42S16160J-6BLI"
+		(property "Value" "IS42S16160J-6BLI-TR"
 			(at 182.4833 63.5 0)
 			(effects
@@
 			(at 162.56 68.58 0)
 			(effects
+				(font
+					(size 1.27 1.27)
+				)
+				(hide yes)
+			)
+		)
+		(property "LCSC Part #" "C2063680"
+			(at 162.56 68.58 0)
+			(effects
