File: hardware/v2.0/cables.kicad_sch (KiCad schematic)
At the start: 2 parts

Commit message: JLCPCB profile
Parts:
- CB1: LCSC Part # (none) -> C454122
- CB2: LCSC Part # (none) -> C7541884
Changed lines of the file:
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@@
 	(title_block
 		(title "GammaPi Zero")
-		(date "2026-02-08")
-		(rev "v2.7.0")
+		(date "2026-02-28")
+		(rev "v2.7.1")
 		(company "Vadym Vikulin, Chengyin Yao (cheyao)")
 		(comment 1 "https://github.com/vikulin/gammapi-zero")
@@
 		)
 		(property "MANUFACTURER" "kinghelm"
+			(at 157.48 81.28 0)
+			(effects
+				(font
+					(size 1.27 1.27)
+				)
+				(hide yes)
+			)
+		)
+		(property "LCSC Part #" "C454122"
 			(at 157.48 81.28 0)
 			(effects
@@
 			(at 157.48 91.44 0)
 			(effects
+				(font
+					(size 1.27 1.27)
+				)
+				(hide yes)
+			)
+		)
+		(property "LCSC Part #" "C7541884"
+			(at 157.48 91.44 0)
+			(effects
