File: hardware/v2.0/dac.kicad_sch (KiCad schematic)
At the start: 7 parts, among them IC3 LM4040AIM3-2.0_NOPB, IC4 LTC2622IMS8#PBF, J8 BM04B-ACHSS-A-GAN-TF_LF__SN_, U1 ECP5U-25F-CABGA256

Commit message: JLCPCB profile
Parts:
- IC3: LCSC Part # (none) -> C2156507
- IC4: LCSC Part # (none) -> C580579
- J8: value BM04B-ACHSS-A-GAN-TF_LF__SN_ -> BM04B-ACHSS-A-GAN-TF(LF)(SN); LCSC Part # (none) -> C5246838
- U1: LCSC Part # (none) -> C1521614
Changed lines of the file:
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@@
 	(title_block
 		(title "GammaPi Zero")
-		(date "2026-02-08")
-		(rev "v2.7.0")
+		(date "2026-02-28")
+		(rev "v2.7.1")
 		(company "Vadym Vikulin, Chengyin Yao (cheyao)")
 		(comment 1 "https://github.com/vikulin/gammapi-zero")
@@
 			)
 		)
+		(property "LCSC Part #" "C580579"
+			(at 158.75 92.71 0)
+			(effects
+				(font
+					(size 1.27 1.27)
+				)
+				(hide yes)
+			)
+		)
 		(pin "8"
 		)
@@
 			)
 		)
+		(property "LCSC Part #" "C2156507"
+			(at 158.75 111.76 0)
+			(effects
+				(font
+					(size 1.27 1.27)
+				)
+				(hide yes)
+			)
+		)
 		(pin "1"
 		)
@@
 			)
 		)
+		(property "LCSC Part #" "C1521614"
+			(at 115.57 105.41 0)
+			(effects
+				(font
+					(size 1.27 1.27)
+				)
+				(hide yes)
+			)
+		)
 		(pin "M5"
 		)
@@
 			)
 		)
-		(property "Value" "BM04B-ACHSS-A-GAN-TF_LF__SN_"
+		(property "Value" "BM04B-ACHSS-A-GAN-TF(LF)(SN)"
 			(at 223.52 105.41 0)
 			(effects
@@
 			(at 212.09 92.71 0)
 			(effects
+				(font
+					(size 1.27 1.27)
+				)
+				(hide yes)
+			)
+		)
+		(property "LCSC Part #" "C5246838"
+			(at 212.09 92.71 0)
+			(effects

Commit message: J8 DAC output connector update
Parts:
- J8: value BM04B-ACHSS-A-GAN-TF(LF)(SN) -> GT-A1201WRS-104B1101; LCSC Part # C5246838 -> C22384775; MANUFACTURER JST Commercial -> G-Switch; MANUFACTURER_PART_NUMBER M04B-ACHSS-A-GAN-TF(LF)(SN) -> GT-A1201WRS-104B1101; Manufacturer_Part_Number BM04B-ACHSS-A-GAN-TF(LF)(SN) -> GT-A1201WRS-104B1101; Mouser Part Number 306-4BACHSSAGANTFL -> (none); Mouser Price/Stock https://www.mouser.co.uk/ProductDetail/JST-Commercial/BM04B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 -> (none)
Changed lines of the file:
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@@
 			)
 		)
-		(property "Value" "BM04B-ACHSS-A-GAN-TF(LF)(SN)"
+		(property "Value" "GT-A1201WRS-104B1101"
 			(at 223.52 105.41 0)
 			(effects
@@
 			)
 		)
-		(property "Datasheet" "https://www.jst-mfg.com/product/pdf/eng/eACH.pdf"
+		(property "Datasheet" "https://www.lcsc.com/datasheet/C22384775.pdf"
 			(at 231.14 287.63 0)
 			(effects
@@
 			)
 		)
-		(property "Description" "CONN HEADER SMD R/A 4POS 1.2MM"
+		(property "Description" "Connector Header 4 position 1.2mm Pitch 1.5A Surface Mount, Right Angle -25℃~+85℃"
 			(at 212.09 92.71 0)
 			(effects
@@
 			)
 		)
-		(property "Mouser Part Number" "306-4BACHSSAGANTFL"
-			(at 231.14 587.63 0)
-			(effects
-				(font
-					(size 1.27 1.27)
-				)
-				(justify left top)
-				(hide yes)
-			)
-		)
-		(property "Mouser Price/Stock" "https://www.mouser.co.uk/ProductDetail/JST-Commercial/BM04B-ACHSS-A-GAN-TFLFSN?qs=QpmGXVUTftFsbdf52tFLQQ%3D%3D"
-			(at 231.14 687.63 0)
-			(effects
-				(font
-					(size 1.27 1.27)
-				)
-				(justify left top)
-				(hide yes)
-			)
-		)
 		(property "Manufacturer_Name" "JST (JAPAN SOLDERLESS TERMINALS)"
 			(at 231.14 787.63 0)
@@
 			)
 		)
-		(property "Manufacturer_Part_Number" "BM04B-ACHSS-A-GAN-TF(LF)(SN)"
+		(property "Manufacturer_Part_Number" "GT-A1201WRS-104B1101"
 			(at 231.14 887.63 0)
 			(effects
@@
 			)
 		)
-		(property "MANUFACTURER" "JST Commercial"
+		(property "MANUFACTURER" "G-Switch"
 			(at 212.09 92.71 0)
 			(effects
@@
 			)
 		)
-		(property "MANUFACTURER_PART_NUMBER" "M04B-ACHSS-A-GAN-TF(LF)(SN)"
+		(property "MANUFACTURER_PART_NUMBER" "GT-A1201WRS-104B1101"
 			(at 212.09 92.71 0)
 			(effects
@@
 			)
 		)
-		(property "LCSC Part #" "C5246838"
+		(property "LCSC Part #" "C22384775"
 			(at 212.09 92.71 0)
 			(effects
