File: hardware/v2.0/io.kicad_sch (KiCad schematic)
At the start: 1 part, among them U1 ECP5U-25F-CABGA256

Commit message: JLCPCB profile
Parts:
- U1: LCSC Part # (none) -> C1521614
Changed lines of the file:
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@@
 	(title_block
 		(title "GammaPi Zero")
-		(date "2026-02-08")
-		(rev "v2.7.0")
+		(date "2026-02-28")
+		(rev "v2.7.1")
 		(company "Vadym Vikulin, Chengyin Yao (cheyao)")
 		(comment 1 "https://github.com/vikulin/gammapi-zero")
@@
 			(at 156.21 93.98 0)
 			(effects
+				(font
+					(size 1.27 1.27)
+				)
+				(hide yes)
+			)
+		)
+		(property "LCSC Part #" "C1521614"
+			(at 156.21 93.98 0)
+			(effects
